File: Sensors/schematic.brd (EAGLE design)
At the start: 55 x 60 mm, 13 parts, among them IC1 LIS331DLHTR, IC2 BMI088, IC3 MCP9803T-M_MS, IC4 MS560702BA03-50

Commit message: Add files via upload
Parts:
- moved R2 72.2 mm to (51.7, 16.0), turned to 180 degrees
- moved R1 61.2 mm to (51.7, 18.7), turned to 180 degrees
- moved C2 59.7 mm to (42.2, 11.7), flipped to the bottom, turned to 180 degrees
- moved C1 56.6 mm to (41.9, 11.4)
- moved C3 49.5 mm to (35.6, 11.4), turned to 180 degrees
- moved C5 46.0 mm to (28.6, 16.4), flipped to the bottom
- moved C4 41.7 mm to (35.6, 11.4), flipped to the bottom
- moved IC4 29.2 mm to (42.2, 15.1), flipped to the bottom, turned to 90 degrees
- moved IC3 17.3 mm to (41.9, 16.5), turned to 270 degrees
- moved IC1 10.9 mm to (35.6, 16.5), turned to 180 degrees
- moved IC2 3.32 mm to (28.7, 16.9), turned to 90 degrees
Connections:
- net 3.3V: now also R1.1, R2.1
- net GND: no longer R1.1, R2.1
Routing:
- net 3.3V: track 0.00 -> 76.1 mm, vias 0 -> 2
- net SDA0: track 0.00 -> 31.1 mm, vias 0 -> 1
- net SCL0: track 0.00 -> 30.4 mm, vias 0 -> 2
- added copper zone on layer 1, net GND
- added copper zone on layer 16, net GND

Commit message: Add files via upload
Parts:
- C4: value 10uF -> 875105240001; device SparkFun-Capacitors:0603-POLAR -> 875105240001:CAPAE430X550N
- moved C4 1.53 mm to (35.4, 9.91), flipped to the top
- moved C1 1.20 mm to (42.3, 12.6), flipped to the bottom
- moved IC3 1.20 mm to (42.3, 17.7), flipped to the bottom
- moved IC4 1.15 mm to (42.0, 16.3), flipped to the top
- moved C2 0.77 mm to (42.0, 12.4), flipped to the top
- moved C3 0.54 mm to (35.2, 11.8), flipped to the bottom, turned to 0 degrees
Connections:
- net 3.3V: now also C4.1; no longer C4.+
- net GND: now also C4.2; no longer C4.-
Routing:
- net SCL0: track 30.4 -> 37.5 mm, vias 2 -> 1
- net 3.3V: track 76.1 -> 80.1 mm
- net SDA0: track 31.1 -> 28.5 mm

Commit message: Add files via upload
Parts:
- added C6: 10uF, SparkFun-Capacitors:0805
- moved C1 9.97 mm to (41.1, 22.5), flipped to the top, turned to 180 degrees
- moved IC3 8.26 mm to (42.5, 25.9), flipped to the top, turned to 180 degrees
- moved C5 3.05 mm to (31.6, 16.4), flipped to the top, turned to 90 degrees
- moved C4 1.52 mm to (35.4, 8.38)
- moved C3 0.77 mm to (35.3, 12.6), flipped to the top, turned to 180 degrees
- moved IC2 0.76 mm to (27.9, 16.9)
Connections:
- net 3.3V: now also C6.1
- net GND: now also C6.2
Routing:
- net SCL0: track 37.5 -> 46.4 mm, vias 1 -> 2
- net 3.3V: track 80.1 -> 82.5 mm, vias 2 -> 3
- net SDA0: track 28.5 -> 30.0 mm, vias 1 -> 0
