File: Sensors/schematic.sch (EAGLE design)
At the start: 13 parts, among them IC1 LIS331DLHTR, IC2 BMI088, IC3 MCP9803T-M_MS, IC4 MS560702BA03-50

Commit message: Add files via upload
Connections:
- net 3.3V: now also R1.1, R2.1
- net GND: no longer R1.1, R2.1
Other:
- moved on the sheet: R1, R2
Changed lines of the file:
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@@
 <part name="C1" library="SparkFun-Capacitors" deviceset="CAP" device="-0805" value="0.1uF"/>
 <part name="C2" library="SparkFun-Capacitors" deviceset="CAP" device="-0805" value="0.1uF"/>
-<part name="GND1" library="supply1" library_urn="urn:adsk.eagle:library:371" deviceset="GND" device=""/>
-<part name="GND2" library="supply1" library_urn="urn:adsk.eagle:library:371" deviceset="GND" device=""/>
 <part name="R2" library="SparkFun-Resistors" deviceset="RESISTOR" device="0805" value="4.7k"/>
 </parts>
@@
 <attribute name="VALUE" x="219.456" y="79.629" size="1.778" layer="96" font="vector"/>
 </instance>
-<instance part="R1" gate="G$1" x="121.92" y="43.18" smashed="yes" rot="R90">
-<attribute name="NAME" x="120.396" y="43.18" size="1.778" layer="95" font="vector" rot="R90" align="bottom-center"/>
-<attribute name="VALUE" x="123.444" y="43.18" size="1.778" layer="96" font="vector" rot="R90" align="top-center"/>
+<instance part="R1" gate="G$1" x="132.08" y="38.1" smashed="yes" rot="R270">
+<attribute name="NAME" x="133.604" y="38.1" size="1.778" layer="95" font="vector" rot="R270" align="bottom-center"/>
+<attribute name="VALUE" x="130.556" y="38.1" size="1.778" layer="96" font="vector" rot="R270" align="top-center"/>
 </instance>
 <instance part="C5" gate="G$1" x="93.98" y="93.98" smashed="yes" rot="R180">
@@
 <attribute name="VALUE" x="155.956" y="157.099" size="1.778" layer="96" font="vector" rot="R180"/>
 </instance>
-<instance part="GND1" gate="1" x="121.92" y="30.48" smashed="yes">
-<attribute name="VALUE" x="119.38" y="27.94" size="1.778" layer="96"/>
-</instance>
-<instance part="GND2" gate="1" x="132.08" y="30.48" smashed="yes">
-<attribute name="VALUE" x="129.54" y="27.94" size="1.778" layer="96"/>
-</instance>
-<instance part="R2" gate="G$1" x="132.08" y="43.18" smashed="yes" rot="R90">
-<attribute name="NAME" x="130.556" y="43.18" size="1.778" layer="95" font="vector" rot="R90" align="bottom-center"/>
-<attribute name="VALUE" x="133.604" y="43.18" size="1.778" layer="96" font="vector" rot="R90" align="top-center"/>
+<instance part="R2" gate="G$1" x="121.92" y="38.1" smashed="yes" rot="R270">
+<attribute name="NAME" x="123.444" y="38.1" size="1.778" layer="95" font="vector" rot="R270" align="bottom-center"/>
+<attribute name="VALUE" x="120.396" y="38.1" size="1.778" layer="96" font="vector" rot="R270" align="top-center"/>
 </instance>
 </instances>
@@
 <wire x1="93.98" y1="96.52" x2="93.98" y2="109.22" width="0.1524" layer="91"/>
 <junction x="93.98" y="109.22"/>
+</segment>
+<segment>
+<pinref part="R2" gate="G$1" pin="1"/>
+<wire x1="121.92" y1="43.18" x2="121.92" y2="48.26" width="0.1524" layer="91"/>
+<label x="121.92" y="48.26" size="1.778" layer="95" rot="R90" xref="yes"/>
+</segment>
+<segment>
+<pinref part="R1" gate="G$1" pin="1"/>
+<junction x="132.08" y="43.18"/>
+<wire x1="132.08" y1="43.18" x2="132.08" y2="48.26" width="0.1524" layer="91"/>
+<label x="132.08" y="48.26" size="1.778" layer="95" rot="R90" xref="yes"/>
 </segment>
 </net>
@@
 <label x="93.98" y="76.2" size="1.778" layer="95" xref="yes"/>
 </segment>
-<segment>
-<pinref part="R1" gate="G$1" pin="1"/>
-<pinref part="GND1" gate="1" pin="GND"/>
-<wire x1="121.92" y1="38.1" x2="121.92" y2="33.02" width="0.1524" layer="91"/>
-</segment>
-<segment>
-<pinref part="R2" gate="G$1" pin="1"/>
-<pinref part="GND2" gate="1" pin="GND"/>
-<wire x1="132.08" y1="38.1" x2="132.08" y2="33.02" width="0.1524" layer="91"/>
-</segment>
 </net>
 <net name="SCL0" class="0">
@@
 <segment>
 <pinref part="R2" gate="G$1" pin="2"/>
-<wire x1="132.08" y1="48.26" x2="132.08" y2="53.34" width="0.1524" layer="91"/>
-<label x="132.08" y="53.34" size="1.778" layer="95" rot="R90" xref="yes"/>
+<wire x1="121.92" y1="33.02" x2="121.92" y2="27.94" width="0.1524" layer="91"/>
+<label x="121.92" y="27.94" size="1.778" layer="95" rot="R270" xref="yes"/>
 </segment>
 </net>
@@
 <segment>
 <pinref part="R1" gate="G$1" pin="2"/>
-<wire x1="121.92" y1="48.26" x2="121.92" y2="53.34" width="0.1524" layer="91"/>
-<label x="121.92" y="53.34" size="1.778" layer="95" rot="R90" xref="yes"/>
-</segment>
-</net>
+<wire x1="132.08" y1="33.02" x2="132.08" y2="27.94" width="0.1524" layer="91"/>
+<label x="132.08" y="27.94" size="1.778" layer="95" rot="R270" xref="yes"/>
+</segment>
+</net>

Commit message: Add files via upload
Parts:
- C4: value 10uF -> 875105240001; device SparkFun-Capacitors:10UF-POLAR-0603-6.3V-20%(TANT) -> 875105240001:875105240001
Changed lines of the file:
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@@
 <part name="IC4" library="MS560702BA03-50" deviceset="MS560702BA03-50" device=""/>
 <part name="FRAME1" library="frames" library_urn="urn:adsk.eagle:library:229" deviceset="LETTER_L" device=""/>
-<part name="C4" library="SparkFun-Capacitors" deviceset="10UF-POLAR" device="-0603-6.3V-20%(TANT)" value="10uF"/>
 <part name="R1" library="SparkFun-Resistors" deviceset="RESISTOR" device="0805" value="4.7k"/>
 <part name="C5" library="SparkFun-Capacitors" deviceset="CAP" device="-0805" value="0.1uF"/>
@@
 <part name="C2" library="SparkFun-Capacitors" deviceset="CAP" device="-0805" value="0.1uF"/>
 <part name="R2" library="SparkFun-Resistors" deviceset="RESISTOR" device="0805" value="4.7k"/>
+<part name="C4" library="875105240001" deviceset="875105240001" device=""/>
 </parts>
 <sheets>
@@
 <attribute name="DRAWING_NAME" x="165.1" y="19.05" size="2.54" layer="94"/>
 </instance>
-<instance part="C4" gate="G$1" x="218.44" y="83.82" smashed="yes">
-<attribute name="NAME" x="219.456" y="84.455" size="1.778" layer="95" font="vector"/>
-<attribute name="VALUE" x="219.456" y="79.629" size="1.778" layer="96" font="vector"/>
-</instance>
 <instance part="R1" gate="G$1" x="132.08" y="38.1" smashed="yes" rot="R270">
 <attribute name="NAME" x="133.604" y="38.1" size="1.778" layer="95" font="vector" rot="R270" align="bottom-center"/>
@@
 <attribute name="NAME" x="123.444" y="38.1" size="1.778" layer="95" font="vector" rot="R270" align="bottom-center"/>
 <attribute name="VALUE" x="120.396" y="38.1" size="1.778" layer="96" font="vector" rot="R270" align="top-center"/>
+</instance>
+<instance part="C4" gate="G$1" x="218.44" y="88.9" smashed="yes" rot="R270">
+<attribute name="NAME" x="224.79" y="80.01" size="1.778" layer="95" rot="R270" align="center-left"/>
+<attribute name="VALUE" x="222.25" y="80.01" size="1.778" layer="96" rot="R270" align="center-left"/>
 </instance>
 </instances>
@@
 <wire x1="218.44" y1="119.38" x2="218.44" y2="99.06" width="0.1524" layer="91"/>
 <junction x="218.44" y="99.06"/>
-<pinref part="C4" gate="G$1" pin="+"/>
-<wire x1="218.44" y1="86.36" x2="218.44" y2="91.44" width="0.1524" layer="91"/>
+<wire x1="218.44" y1="86.36" x2="218.44" y2="88.9" width="0.1524" layer="91"/>
+<wire x1="218.44" y1="88.9" x2="218.44" y2="91.44" width="0.1524" layer="91"/>
 <wire x1="218.44" y1="91.44" x2="213.36" y2="91.44" width="0.1524" layer="91"/>
 <wire x1="213.36" y1="91.44" x2="208.28" y2="91.44" width="0.1524" layer="91"/>
@@
 <junction x="213.36" y="91.44"/>
 <pinref part="C3" gate="G$1" pin="2"/>
+<pinref part="C4" gate="G$1" pin="+"/>
+<junction x="218.44" y="88.9"/>
 </segment>
 <segment>
@@
 <wire x1="228.6" y1="66.04" x2="213.36" y2="66.04" width="0.1524" layer="91"/>
 <wire x1="213.36" y1="66.04" x2="187.96" y2="66.04" width="0.1524" layer="91"/>
-<pinref part="C4" gate="G$1" pin="-"/>
-<wire x1="218.44" y1="78.74" x2="218.44" y2="73.66" width="0.1524" layer="91"/>
+<wire x1="218.44" y1="78.74" x2="218.44" y2="76.2" width="0.1524" layer="91"/>
+<wire x1="218.44" y1="76.2" x2="218.44" y2="73.66" width="0.1524" layer="91"/>
 <wire x1="218.44" y1="73.66" x2="213.36" y2="73.66" width="0.1524" layer="91"/>
 <wire x1="213.36" y1="73.66" x2="208.28" y2="73.66" width="0.1524" layer="91"/>
@@
 <pinref part="C3" gate="G$1" pin="1"/>
 <wire x1="208.28" y1="78.74" x2="208.28" y2="73.66" width="0.1524" layer="91"/>
-</segment>
-<segment>
+<pinref part="C4" gate="G$1" pin="-"/>
+<junction x="218.44" y="76.2"/>
+</segment>
+<segment>

Commit message: Add files via upload
Parts:
- added C6: 10uF, SparkFun-Capacitors:10UF-0805-10V-10%
Connections:
- net 3.3V: now also C6.1
- net GND: now also C6.2
Other:
- moved on the sheet: R1, R2
Changed lines of the file:
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@@
 <part name="R2" library="SparkFun-Resistors" deviceset="RESISTOR" device="0805" value="4.7k"/>
 <part name="C4" library="875105240001" deviceset="875105240001" device=""/>
+<part name="C6" library="SparkFun-Capacitors" deviceset="10UF" device="-0805-10V-10%" value="10uF"/>
 </parts>
 <sheets>
@@
 <attribute name="DRAWING_NAME" x="165.1" y="19.05" size="2.54" layer="94"/>
 </instance>
-<instance part="R1" gate="G$1" x="132.08" y="38.1" smashed="yes" rot="R270">
-<attribute name="NAME" x="133.604" y="38.1" size="1.778" layer="95" font="vector" rot="R270" align="bottom-center"/>
-<attribute name="VALUE" x="130.556" y="38.1" size="1.778" layer="96" font="vector" rot="R270" align="top-center"/>
+<instance part="R1" gate="G$1" x="139.7" y="38.1" smashed="yes" rot="R270">
+<attribute name="NAME" x="143.764" y="38.1" size="1.778" layer="95" font="vector" rot="R270" align="bottom-center"/>
+<attribute name="VALUE" x="138.176" y="38.1" size="1.778" layer="96" font="vector" rot="R270" align="top-center"/>
 </instance>
 <instance part="C5" gate="G$1" x="93.98" y="93.98" smashed="yes" rot="R180">
@@
 <attribute name="VALUE" x="155.956" y="157.099" size="1.778" layer="96" font="vector" rot="R180"/>
 </instance>
-<instance part="R2" gate="G$1" x="121.92" y="38.1" smashed="yes" rot="R270">
-<attribute name="NAME" x="123.444" y="38.1" size="1.778" layer="95" font="vector" rot="R270" align="bottom-center"/>
-<attribute name="VALUE" x="120.396" y="38.1" size="1.778" layer="96" font="vector" rot="R270" align="top-center"/>
+<instance part="R2" gate="G$1" x="129.54" y="38.1" smashed="yes" rot="R270">
+<attribute name="NAME" x="131.064" y="38.1" size="1.778" layer="95" font="vector" rot="R270" align="bottom-center"/>
+<attribute name="VALUE" x="128.016" y="38.1" size="1.778" layer="96" font="vector" rot="R270" align="top-center"/>
 </instance>
 <instance part="C4" gate="G$1" x="218.44" y="88.9" smashed="yes" rot="R270">
 <attribute name="NAME" x="224.79" y="80.01" size="1.778" layer="95" rot="R270" align="center-left"/>
 <attribute name="VALUE" x="222.25" y="80.01" size="1.778" layer="96" rot="R270" align="center-left"/>
+</instance>
+<instance part="C6" gate="G$1" x="116.84" y="38.1" smashed="yes">
+<attribute name="NAME" x="118.364" y="41.021" size="1.778" layer="95" font="vector"/>
+<attribute name="VALUE" x="118.364" y="35.941" size="1.778" layer="96" font="vector"/>
 </instance>
 </instances>
@@
 <segment>
 <pinref part="R2" gate="G$1" pin="1"/>
-<wire x1="121.92" y1="43.18" x2="121.92" y2="48.26" width="0.1524" layer="91"/>
-<label x="121.92" y="48.26" size="1.778" layer="95" rot="R90" xref="yes"/>
+<wire x1="129.54" y1="43.18" x2="129.54" y2="48.26" width="0.1524" layer="91"/>
+<label x="129.54" y="48.26" size="1.778" layer="95" rot="R90" xref="yes"/>
 </segment>
 <segment>
 <pinref part="R1" gate="G$1" pin="1"/>
-<junction x="132.08" y="43.18"/>
-<wire x1="132.08" y1="43.18" x2="132.08" y2="48.26" width="0.1524" layer="91"/>
-<label x="132.08" y="48.26" size="1.778" layer="95" rot="R90" xref="yes"/>
+<junction x="139.7" y="43.18"/>
+<wire x1="139.7" y1="43.18" x2="139.7" y2="48.26" width="0.1524" layer="91"/>
+<label x="139.7" y="48.26" size="1.778" layer="95" rot="R90" xref="yes"/>
+</segment>
+<segment>
+<pinref part="C6" gate="G$1" pin="1"/>
+<wire x1="116.84" y1="43.18" x2="116.84" y2="48.26" width="0.1524" layer="91"/>
+<label x="116.84" y="48.26" size="1.778" layer="95" rot="R90" xref="yes"/>
 </segment>
 </net>
@@
 <label x="93.98" y="76.2" size="1.778" layer="95" xref="yes"/>
 </segment>
+<segment>
+<pinref part="C6" gate="G$1" pin="2"/>
+<wire x1="116.84" y1="35.56" x2="116.84" y2="27.94" width="0.1524" layer="91"/>
+<label x="116.84" y="27.94" size="1.778" layer="95" rot="R270" xref="yes"/>
+</segment>
 </net>
 <net name="SCL0" class="0">
@@
 <segment>
 <pinref part="R2" gate="G$1" pin="2"/>
-<wire x1="121.92" y1="33.02" x2="121.92" y2="27.94" width="0.1524" layer="91"/>
-<label x="121.92" y="27.94" size="1.778" layer="95" rot="R270" xref="yes"/>
+<wire x1="129.54" y1="33.02" x2="129.54" y2="27.94" width="0.1524" layer="91"/>
+<label x="129.54" y="27.94" size="1.778" layer="95" rot="R270" xref="yes"/>
 </segment>
 </net>
@@
 <segment>
 <pinref part="R1" gate="G$1" pin="2"/>
-<wire x1="132.08" y1="33.02" x2="132.08" y2="27.94" width="0.1524" layer="91"/>
-<label x="132.08" y="27.94" size="1.778" layer="95" rot="R270" xref="yes"/>
-</segment>
-</net>
+<wire x1="139.7" y1="33.02" x2="139.7" y2="27.94" width="0.1524" layer="91"/>
+<label x="139.7" y="27.94" size="1.778" layer="95" rot="R270" xref="yes"/>
+</segment>
+</net>
