File: STM32L433 MCU board/schematic.brd (EAGLE design)
At the start: 55 x 60 mm, 28 parts, among them T1 2N2222, U2 STM32L476RCT6, Y2 ABS25-32.768KHZ-6-T, Y3 ECS-160-S-5PX-TR

Commit message: Added logo
Routing:
- net GND: vias 125 -> 127
Other:
- board text added: "C:/Users/callu/Documents/UBC Rocket/2022 Avionics/image_monochrome.bmp"
